Commit message: added hazard level boxes

File: resources/objects/obstacle.urdf (robot description, URDF)
Before this commit: robot box, 1 links, 0 joints
Links:
- link box: geometry collision box size=.25 .25 .25; visual box size=.25 .25 .25

Commit message: updated path plan visualization to include bounding box

File: resources/objects/obstacle.urdf (robot description, URDF)
Before this commit: robot box, 1 links, 0 joints
Links:
- link box: geometry collision box size=1 1 1; visual box size=1 1 1
